Commit message: Minor changes

File: resources/base.urdf (robot description, URDF)
Before this commit: robot base, 1 links, 0 joints
Links:
- link base_link: geometry collision box size=2 4 0.01; visual box size=2 4 0.01

File: resources/ramp.urdf (robot description, URDF)
Before this commit: robot ramp, 1 links, 0 joints
Links:
- link base_link: geometry collision box size=2 4 0.01; visual box size=2 4 0.01

Commit message: Created branch for laboratory

File: resources/base.urdf (robot description, URDF)
Before this commit: robot base, 1 links, 0 joints
Links:
- link base_link: geometry collision box size=2 2 0.01; visual box size=2 2 0.01
