Commit message: RGB images taken on oct 13

File: resources/urdf/ramp_2.urdf (robot description, URDF)
Before this commit: robot ramp, 1 links, 0 joints
Links:
- link base_link: geometry collision box size=2 2 0.01; visual box size=2 2 0.01

File: resources/urdf/ramp_3.urdf (robot description, URDF)
Before this commit: robot ramp, 1 links, 0 joints
Links:
- link base_link: geometry collision box size=2 3 0.01; visual box size=2 3 0.01

File: resources/urdf/ramp_4.urdf (robot description, URDF)
Before this commit: robot ramp, 1 links, 0 joints
Links:
- link base_link: geometry collision box size=2 4 0.01; visual box size=2 4 0.01

Commit message: Added more rgb images

File: resources/urdf/ramp_2.urdf (robot description, URDF)
Before this commit: robot ramp, 1 links, 0 joints
Links:
- link base_link: geometry collision box size=1.5 2 0.01; visual box size=1.5 2 0.01

File: resources/urdf/ramp_3.urdf (robot description, URDF)
Before this commit: robot ramp, 1 links, 0 joints
Links:
- link base_link: geometry collision box size=1.5 3 0.01; visual box size=1.5 3 0.01

File: resources/urdf/ramp_4.urdf (robot description, URDF)
Before this commit: robot ramp, 1 links, 0 joints
Links:
- link base_link: geometry collision box size=1.5 4 0.01; visual box size=1.5 4 0.01
