Commit message: Newest commit

File: resources/urdf/bridge.urdf (robot description, URDF)
Before this commit: robot bridge, 1 links, 0 joints
Links:
- link base_link: geometry collision box size=2 20 0.01; visual box size=2 20 0.01

Commit message: Added new experiments of varying max frequency and using bridge env

File: resources/urdf/bridge.urdf (robot description, URDF)
Before this commit: robot bridge, 1 links, 0 joints
Links:
- link base_link: geometry collision box size=2 100 0.01; visual box size=2 100 0.01
